Commit message: Partially implemented Gazebo simulation

File: rpi_workspace/src/robot_description/urdf/slam_robot.urdf.xacro (robot description, xacro)
@@ -1,5 +1,12 @@
 <?xml version="1.0"?>
 <robot name="slam_robot" xmlns:xacro="http://www.ros.org/wiki/xacro">
-  <!-- Define some colors for visualization -->
+  <!-- Define properties -->
+  <xacro:property name="base_width" value="0.20"/>
+  <xacro:property name="base_length" value="0.25"/>
+  <xacro:property name="base_height" value="0.10"/>
+  <xacro:property name="wheel_radius" value="0.04"/>
+  <xacro:property name="wheel_width" value="0.02"/>
+  <xacro:property name="wheel_separation" value="0.22"/>
+  <!-- Define materials for RViz -->
   <material name="blue">
     <color rgba="0.2 0.3 0.8 1.0"/>
@@ -14,97 +21,299 @@
     <color rgba="0.5 0.5 0.5 1.0"/>
   </material>
-  <!-- Base link (robot center/main body) -->
+  <material name="black">
+    <color rgba="0.1 0.1 0.1 1.0"/>
+  </material>
+  <!-- Base link (robot main body) -->
   <link name="base_link">
     <visual>
       <geometry>
-        <box size="0.25 0.20 0.10"/>  <!-- 25cm x 20cm x 10cm robot body -->
-      </geometry>
-      <origin xyz="0 0 0.05" rpy="0 0 0"/>  <!-- Centered at half height -->
+        <box size="${base_length} ${base_width} ${base_height}"/>
+      </geometry>
+      <origin xyz="0 0 ${base_height/2}" rpy="0 0 0"/>
       <material name="blue"/>
     </visual>
     <collision>
       <geometry>
-        <box size="0.25 0.20 0.10"/>
-      </geometry>
-      <origin xyz="0 0 0.05" rpy="0 0 0"/>
-    </collision>
-    <inertial>
-      <mass value="1.0"/>
-      <inertia ixx="0.01" ixy="0.0" ixz="0.0" iyy="0.01" iyz="0.0" izz="0.01"/>
-    </inertial>
-  </link>
+        <box size="${base_length} ${base_width} ${base_height}"/>
+      </geometry>
+      <origin xyz="0 0 ${base_height/2}" rpy="0 0 0"/>
+    </collision>
+    <inertial>
+      <mass value="2.0"/>
+      <origin xyz="0 0 ${base_height/2}" rpy="0 0 0"/>
+      <inertia ixx="0.0167" ixy="0.0" ixz="0.0" iyy="0.0208" iyz="0.0" izz="0.0292"/>
+    </inertial>
+  </link>
+  <!-- Gazebo material for base_link -->
+  <gazebo reference="base_link">
+    <material>Gazebo/Blue</material>
+  </gazebo>
   <!-- IMU link -->
   <link name="imu_link">
     <visual>
       <geometry>
-        <box size="0.02 0.02 0.01"/>  <!-- Small box representing IMU -->
+        <box size="0.02 0.02 0.01"/>
       </geometry>
       <material name="red"/>
     </visual>
+    <inertial>
+      <mass value="0.01"/>
+      <inertia ixx="0.00001" ixy="0.0" ixz="0.0" iyy="0.00001" iyz="0.0" izz="0.00001"/>
+    </inertial>
   </link>
   <joint name="base_to_imu" type="fixed">
     <parent link="base_link"/>
     <child link="imu_link"/>
-    <!-- IMU mounted at center of robot, 6cm above base -->
     <origin xyz="0.0 0.0 0.11" rpy="0 0 0"/>
   </joint>
+<gazebo reference="imu_link">
+    <material>Gazebo/Red</material>
+  </gazebo>
+  <!-- IMU Sensor Plugin - ADD THIS -->
+  <gazebo reference="imu_link">
+    <sensor name="imu_sensor" type="imu">
+      <always_on>true</always_on>
+      <update_rate>100</update_rate>
+      <imu>
+        <angular_velocity>
+          <x>
+            <noise type="gaussian">
+              <mean>0.0</mean>
+              <stddev>0.01</stddev>
+            </noise>
+          </x>
+          <y>
+            <noise type="gaussian">
+              <mean>0.0</mean>
+              <stddev>0.01</stddev>
+            </noise>
+          </y>
+          <z>
+            <noise type="gaussian">
+              <mean>0.0</mean>
+              <stddev>0.01</stddev>
+            </noise>
+          </z>
+        </angular_velocity>
+        <linear_acceleration>
+          <x>
+            <noise type="gaussian">
+              <mean>0.0</mean>
+              <stddev>0.05</stddev>
+            </noise>
+          </x>
+          <y>
+            <noise type="gaussian">
+              <mean>0.0</mean>
+              <stddev>0.05</stddev>
+            </noise>
+          </y>
+          <z>
+            <noise type="gaussian">
+              <mean>0.0</mean>
+              <stddev>0.05</stddev>
+            </noise>
+          </z>
+        </linear_acceleration>
+      </imu>
+    </sensor>
+  </gazebo>
   <!-- Camera link -->
   <link name="camera_link">
     <visual>
       <geometry>
-        <box size="0.025 0.025 0.025"/>  <!-- Pi Camera V2 approximate size -->
+        <box size="0.025 0.025 0.025"/>
       </geometry>
       <material name="green"/>
     </visual>
+    <inertial>
+      <mass value="0.01"/>
+      <inertia ixx="0.00001" ixy="0.0" ixz="0.0" iyy="0.00001" iyz="0.0" izz="0.00001"/>
+    </inertial>
   </link>
   <joint name="base_to_camera" type="fixed">
     <parent link="base_link"/>
     <child link="camera_link"/>
-    <!-- Camera mounted at front of robot, 8cm above base, facing forward -->
     <origin xyz="0.125 0.0 0.13" rpy="0 0 0"/>
   </joint>
+  <gazebo reference="camera_link">
+    <material>Gazebo/Green</material>
+  </gazebo>
+  <!-- Camera Sensor -->
+  <gazebo reference="camera_link">
+    <sensor name="camera_sensor" type="camera">
+      <update_rate>30</update_rate>
+      <always_on>1</always_on>
+      <visualize>true</visualize>
+      <camera>
+        <horizontal_fov>1.085</horizontal_fov>
+        <image>
+          <width>640</width>
+          <height>480</height>
+          <format>R8G8B8</format>
+        </image>
+        <clip>
+          <near>0.1</near>
+          <far>100</far>
+        </clip>
+        <noise>
+          <type>gaussian</type>
+          <mean>0.0</mean>
+          <stddev>0.007</stddev>
+        </noise>
+      </camera>
+    </sensor>
+  </gazebo>
   <!-- LiDAR link -->
   <link name="laser_link">
     <visual>
       <geometry>
-        <cylinder radius="0.035" length="0.04"/>  <!-- Cylindrical LiDAR -->
+        <cylinder radius="0.035" length="0.04"/>
       </geometry>
       <material name="gray"/>
     </visual>
+    <collision>
+      <geometry>
+        <cylinder radius="0.035" length="0.04"/>
+      </geometry>
+    </collision>
+    <inertial>
+      <mass value="0.2"/>
+      <inertia ixx="0.0001" ixy="0.0" ixz="0.0" iyy="0.0001" iyz="0.0" izz="0.0001"/>
+    </inertial>
   </link>
   <joint name="base_to_laser" type="fixed">
     <parent link="base_link"/>
     <child link="laser_link"/>
-    <!-- LiDAR mounted at top center of robot, 15cm above base -->
     <origin xyz="0.0 0.0 0.15" rpy="0 0 0"/>
   </joint>
-  <!-- Optional: Add wheels for visualization (non-functional) -->
+  <gazebo reference="laser_link">
+    <material>Gazebo/Gray</material>
+  </gazebo>
+  <!-- LiDAR Sensor -->
+  <gazebo reference="laser_link">
+    <sensor name="lidar_sensor" type="ray">
+      <always_on>true</always_on>
+      <update_rate>10</update_rate>
+      <visualize>true</visualize>
+      <ray>
+        <scan>
+          <horizontal>
+            <samples>360</samples>
+            <resolution>1</resolution>
+            <min_angle>-3.14159</min_angle>
+            <max_angle>3.14159</max_angle>
+          </horizontal>
+        </scan>
+        <range>
+          <min>0.1</min>
+          <max>10.0</max>
+          <resolution>0.01</resolution>
+        </range>
+        <noise>
+          <type>gaussian</type>
+          <mean>0.0</mean>
+          <stddev>0.01</stddev>
+        </noise>
+      </ray>
+    </sensor>
+  </gazebo>
+  <!-- Left wheel -->
   <link name="left_wheel">
     <visual>
       <geometry>
-        <cylinder radius="0.04" length="0.02"/>
-      </geometry>
-      <origin xyz="0 0 0" rpy="1.5708 0 0"/>  <!-- Rotate 90 degrees -->
-      <material name="gray"/>
-    </visual>
-  </link>
-  <joint name="base_to_left_wheel" type="fixed">
+        <cylinder radius="${wheel_radius}" length="${wheel_width}"/>
+      </geometry>
+      <origin xyz="0 0 0" rpy="1.5708 0 0"/>
+      <material name="black"/>
+    </visual>
+    <collision>
+      <geometry>
+        <cylinder radius="${wheel_radius}" length="${wheel_width}"/>
+      </geometry>
+      <origin xyz="0 0 0" rpy="1.5708 0 0"/>
+    </collision>
+    <inertial>
+      <mass value="0.1"/>
+      <origin xyz="0 0 0" rpy="1.5708 0 0"/>
+      <inertia ixx="0.0001" ixy="0.0" ixz="0.0" iyy="0.0001" iyz="0.0" izz="0.0001"/>
+    </inertial>
+  </link>
+  <joint name="base_to_left_wheel" type="continuous">
     <parent link="base_link"/>
     <child link="left_wheel"/>
-    <origin xyz="0.0 0.11 0.04" rpy="0 0 0"/>  <!-- Left side -->
-  </joint>
+    <origin xyz="0.0 ${wheel_separation/2} ${wheel_radius}" rpy="0 0 0"/>
+    <axis xyz="0 1 0"/>
+  </joint>
+  <gazebo reference="left_wheel">
+    <material>Gazebo/Black</material>
+  </gazebo>
+  <!-- Right wheel -->
   <link name="right_wheel">
     <visual>
       <geometry>
-        <cylinder radius="0.04" length="0.02"/>
-      </geometry>
-      <origin xyz="0 0 0" rpy="1.5708 0 0"/>
-      <material name="gray"/>
-    </visual>
-  </link>
-  <joint name="base_to_right_wheel" type="fixed">
+        <cylinder radius="${wheel_radius}" length="${wheel_width}"/>
+      </geometry>
+      <origin xyz="0 0 0" rpy="1.5708 0 0"/>
+      <material name="black"/>
+    </visual>
+    <collision>
+      <geometry>
+        <cylinder radius="${wheel_radius}" length="${wheel_width}"/>
+      </geometry>
+      <origin xyz="0 0 0" rpy="1.5708 0 0"/>
+    </collision>
+    <inertial>
+      <mass value="0.1"/>
+      <origin xyz="0 0 0" rpy="1.5708 0 0"/>
+      <inertia ixx="0.0001" ixy="0.0" ixz="0.0" iyy="0.0001" iyz="0.0" izz="0.0001"/>
+    </inertial>
+  </link>
+  <joint name="base_to_right_wheel" type="continuous">
     <parent link="base_link"/>
     <child link="right_wheel"/>
-    <origin xyz="0.0 -0.11 0.04" rpy="0 0 0"/>  <!-- Right side -->
-  </joint>
+    <origin xyz="0.0 ${-wheel_separation/2} ${wheel_radius}" rpy="0 0 0"/>
+    <axis xyz="0 1 0"/>
+  </joint>
+  <gazebo reference="right_wheel">
+    <material>Gazebo/Black</material>
+  </gazebo>
+  <!-- Caster wheel (front) for stability -->
+  <link name="caster_wheel">
+    <visual>
+      <geometry>
+        <sphere radius="0.02"/>
+      </geometry>
+      <material name="black"/>
+    </visual>
+    <collision>
+      <geometry>
+        <sphere radius="0.02"/>
+      </geometry>
+    </collision>
+    <inertial>
+      <mass value="0.05"/>
+      <inertia ixx="0.00001" ixy="0.0" ixz="0.0" iyy="0.00001" iyz="0.0" izz="0.00001"/>
+    </inertial>
+  </link>
+  <joint name="base_to_caster" type="fixed">
+    <parent link="base_link"/>
+    <child link="caster_wheel"/>
+    <origin xyz="0.10 0.0 0.02" rpy="0 0 0"/>
+  </joint>
+  <gazebo reference="caster_wheel">
+    <material>Gazebo/Black</material>
+    <mu1>0.0</mu1>  <!-- Frictionless caster -->
+    <mu2>0.0</mu2>
+  </gazebo>
+  <!-- Differential Drive Plugin -->
+  <gazebo>
+    <plugin filename="libgz-sim-diff-drive-system.so" name="gz::sim::systems::DiffDrive">
+      <left_joint>base_to_left_wheel</left_joint>
+      <right_joint>base_to_right_wheel</right_joint>
+      <wheel_separation>${wheel_separation}</wheel_separation>
+      <wheel_radius>${wheel_radius}</wheel_radius>
+      <odom_publish_frequency>50</odom_publish_frequency>
+    </plugin>
+  </gazebo>
 </robot>
